Commit message: Minor change, now velodyne works in Gazebo sim

File: hector_sensors_description/urdf/vlp16.urdf.xacro (robot description, xacro)
@@ -9,5 +9,5 @@
       </joint>
       <link name="${name}_frame">
-        <xacro:inertial_sphere mass="0.83" diameter="0.1033" />
+        <xacro:macro name="inertial_sphere" mass="0.83" diameter="0.1033" />
         <!-- Visual geometry by velodyne_simulator https://bitbucket.org/DataspeedInc/velodyne_simulator -->
         <visual>
